File: kicad_files/BattleSync.kicad_sch (KiCad schematic)
At the start: 14 parts, among them SW1 SW_SPDT, U1 113991054, U2 DFR0299

Commit message: Update PCB design with footprint and net changes
Hardware design updates including:
- Revised net numbering and routing
- Footprint changes (connector and capacitor updates)
- Added Seeeduino XIAO ESP32S3 KiCAD library
- Updated component placement and connections

These changes align the PCB design with the ESP32-S3 hardware migration.

🤖 Generated with [Claude Code](https://claude.com/claude-code)

Co-Authored-By: Claude <noreply@anthropic.com>
Parts:
- removed BT1: Battery_Cell, Connector_JST:JST_PH_B2B-PH-K_1x02_P2.00mm_Vertical, symbol Device:Battery_Cell
- added BT2: Battery_Cell, Connector_JST:JST_PH_B2B-PH-K_1x02_P2.00mm_Vertical, symbol Device:Battery_Cell
- added C1: C_Polarized, Capacitor_THT:CP_Radial_D4.0mm_P2.00mm, symbol Device:C_Polarized
- D1, D2, D3, D4, D5, D6, D7, D8, SW1: footprint Connector_JST:JST_PH_B2B-PH-K_1x02_P2.00mm_Vertical -> Connector_Wire:SolderWire-0.1sqmm_1x02_P3.6mm_D0.4mm_OD1mm
- D9: footprint Connector_JST:JST_PH_B2B-PH-K_1x02_P2.00mm_Vertical -> Connector_Wire:SolderWire-0.1sqmm_1x03_P3.6mm_D0.4mm_OD1mm; symbol Device:LED -> LED:WS2812B
- U1: value 113991054 -> ESP32-S3; footprint Seeeduino xiao ESP32C3 KiCAD Library:MODULE_113991054 -> RF_Module:MCU_Seeed_ESP32C3
Connections:
- net at D1.1 (K), D2.1 (K), D3.1 (K)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: now also D9.3 (VSS), BT2.2 (-), C1.2; no longer D9.1 (K)
- net at SW1.1 (A), U1.15 (BAT), U2.1 (VCC): now also C1.1
- net at SW1.2 (B): now also BT2.1 (+)
- net at D9.2 (DOUT): no longer U1.11 (GPIO10_D10_MOSI)
- net at U1.12 (3V3): now also D9.1 (VDD)
- new net: D9.4 (DIN), U1.11 (GPIO10_D10_MOSI)
